File: FreeServoProject.sch (KiCad schematic (older format))
At the start: 48 parts, among them J1 Conn_01x03, J2 Conn_01x03, J3 Conn_01x03, J4 Conn_01x03, M1 Motor_DC, U1 AP7381-33Y-13, U2 STM32F303K8Tx, U3 VNH7070BASTR, U4 74LVC1G125, U5 74LVC1G126, U6 ST1480ACDR, U7 AS5600-ASOM

Commit message: update
Parts:
- C1: value 1u -> 1u 38V
- J1: value Conn_01x03 -> Conthrough; symbol Connector_Generic:Conn_01x03 -> Connector_Generic:Conn_01x04; #manf (none) -> XB-3-6-4P; order_URL (none) -> https://akizukidenshi.com/catalog/g/gC-15594/
- R1, R13, R14, R2, R7: footprint (none) -> Resistors_SMD:R_0603; #manf (none) -> CRG0603F10K/10; order_URL (none) -> https://www.digikey.jp/product-detail/ja/te-connectivity-pa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
Connections:
- net +3V3: now also J1.4 (Pin_4), U2.1 (VDD), U2.17 (VDD)
- net GND: no longer FB1.2, U2.1 (VDD), U2.17 (VDD), U2.5 (VDDA)
- net Potentiometer: now also U2.9 (PA3); no longer U2.14 (PB0)
- new net: FB1.2, U2.5 (VDDA)
Other:
- moved on the sheet: C15, C3, C4, C5, C6, C7, C8, FB1, R1, U2

Commit message: Add files via upload
フットプリント追加と基板設計前。
Parts:
- added C17, C18, C19, C20, C21: 10u35V, Capacitors_SMD:C_0603, symbol Device:C
- added R15: 10k, Resistors_SMD:R_0603, symbol Device:R
- C1: value 1u 38V -> 1u35V; footprint (none) -> Capacitors_SMD:C_0603; #manf (none) -> UMK107BJ105KA-T; order_URL (none) -> https://www.digikey.jp/product-detail/ja/taiyo-yuden/UMK107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
- C10: footprint (none) -> Capacitors_SMD:C_0603; #manf (none) -> 0603B333K500CT; order_URL (none) -> https://www.digikey.jp/product-detail/ja/walsin-technology-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
- C11: value 220u 38V -> 220u35V; footprint (none) -> Capacitors_ThroughHole:CP_Radial_D8.0mm_P3.50mm; #manf (none) -> 35ZLH220MEFCCT8X11.5
- C14, C15, C16, C4, C5, C7, C8, C9: footprint (none) -> Capacitors_SMD:C_0603; #manf (none) -> C0603C104M4RACTU; order_URL (none) -> https://www.digikey.jp/product-detail/ja/kemet/C0603C104M4R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
- C2: footprint (none) -> Capacitors_SMD:C_0603; #manf (none) -> CL10A225KQ8NNNC; order_URL (none) -> https://www.digikey.jp/product-detail/ja/samsung-electro-me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
- C3: footprint (none) -> Capacitors_SMD:C_0603; #manf (none) -> CL10B105MO8NNWC; order_URL (none) -> https://www.digikey.jp/product-detail/ja/samsung-electro-me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
- C6: footprint (none) -> Capacitors_SMD:C_0603; #manf (none) -> 0603B103K500CT; order_URL (none) -> https://www.digikey.jp/product-detail/ja/walsin-technology-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
- D1: footprint (none) -> LEDs:LED_0603; #manf (none) -> LS Q976-NR-1; order_URL (none) -> https://www.digikey.jp/product-detail/ja/osram-opto-semicon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
- FB1: footprint (none) -> Capacitors_SMD:C_0603; #manf (none) -> BLM18BD102SN1D; order_URL (none) -> https://www.digikey.jp/product-detail/ja/murata-electronics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
- J1: value Conthrough -> 4P-SBN; footprint (none) -> 4P-SBN:4P-SBN; #manf XB-3-6-4P -> 4P-SBN; order_URL https://akizukidenshi.com/catalog/g/gC-15594/ -> https://order.jst-mfg.com/InternetShop/app/index?back=2&pro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
- J2: footprint (none) -> Pin_Headers:Pin_Header_Straight_1x03_Pitch2.54mm
- J3: value Conn_01x03 -> Conn_01x04; footprint (none) -> Connectors_JST:JST_EH_B4B-EH-A_1x04_P2.50mm_Vertical
- J4: value Conn_01x03 -> Conn_01x04; footprint (none) -> Pin_Headers:Pin_Header_Straight_1x04_Pitch2.54mm
- M1: footprint (none) -> Pin_Headers:Pin_Header_Straight_1x02_Pitch2.54mm
- R1, R12, R13, R14, R2, R7: #manf CRG0603F10K/10 -> ‎RC0603JR-0710KL‎; order_URL https://www.digikey.jp/product-detail/ja/te-connectivity-pa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 -> https://www.digikey.jp/product-detail/ja/yageo/RC0603JR-071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
- R10, R5, R6, R9: footprint (none) -> Resistors_SMD:R_0603; #manf (none) -> CRGCQ0603F1K0; order_URL (none) -> https://www.digikey.jp/product-detail/ja/te-connectivity-pa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
- R11, R3: footprint (none) -> Resistors_SMD:R_0603; #manf (none) -> CRGCQ0603F6K8; order_URL (none) -> https://www.digikey.jp/product-detail/ja/te-connectivity-pa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
- R4: footprint (none) -> Resistors_SMD:R_0603; #manf (none) -> RC0603FR-07910RL; order_URL (none) -> https://www.digikey.jp/product-detail/ja/yageo/RC0603FR-079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
- R8: footprint (none) -> Resistors_SMD:R_0603; #manf (none) -> RC0603FR-071K5L; order_URL (none) -> https://www.digikey.jp/product-detail/ja/yageo/RC0603FR-071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
- RV1: value R_POT -> RDC503052A; footprint (none) -> RDC503052A:RDC503052A; #manf (none) -> RDC503052A; order_URL (none) -> https://www.mouser.jp/ProductDetail/Alps-Alpine/RDC503052A?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
- U2: footprint Package_QFP:LQFP-32_7x7mm_P0.8mm -> Housings_QFP:LQFP-32_7x7mm_Pitch0.8mm
- U6: footprint Package_SO:SOIC-8_3.9x4.9mm_P1.27mm -> Housings_SOIC:SOIC-8_3.9x4.9mm_Pitch1.27mm
Connections:
- net +3V3: now also R15.2; no longer C1.1, C11.1, J1.4 (Pin_4), J2.2 (Pin_2), J3.2 (Pin_2), R3.1, U1.3 (VIN), U3.12 (VCC), U3.4 (VCC), U3.5 (VCC)
- net GND: now also C17.2, C18.2, C19.2, C20.2, C21.2
- new net +BATT: C1.1, C11.1, C17.1, C18.1, C19.1, C20.1, C21.1, J2.2 (Pin_2), J3.2 (Pin_2), R3.1, U1.3 (VIN), U3.12 (VCC), U3.4 (VCC), U3.5 (VCC)
- new net RST: J1.4 (Pin_4), R15.1
Other:
- moved on the sheet: C16, RV1

Commit message: Add files via upload
Parts:
- added C22: 10u35V, Capacitors_SMD:C_1210, symbol Device:C
- added H1, H2, H3, H4: MountingHole_Pad, Wire_Pads:SolderWirePad_single_2mmDrill, symbol Mechanical:MountingHole_Pad
- added J10: Conn_01x04, Connect:Grove_1x04, symbol Connector_Generic:Conn_01x04
- added J11: S3B-PH-K, Connectors_JST:JST_PH_S3B-PH-K_1x03_P2.00mm_Horizontal, symbol Connector_Generic:Conn_01x03
- added J12: 5_SMD_Pad, SMD_Pad:5_SMD_Pad, symbol Connector_Generic:Conn_01x05
- added J5, J6: Pin_Header_Straight_1x04_Pitch2.00mm, Pin_Headers:Pin_Header_Straight_1x04_Pitch2.00mm, symbol Connector_Generic:Conn_01x04
- added J7, J8: Socket_Strip_Straight_1x04_Pitch2.00mm, Socket_Strips:Socket_Strip_Straight_1x04_Pitch2.00mm, symbol Connector_Generic:Conn_01x04
- added J9: Conn_01x04, Connectors_JST:JST_EH_B4B-EH-A_1x04_P2.50mm_Vertical, symbol Connector_Generic:Conn_01x04
- added Y1: Resonator, CSTNE8M00G55Z000R0:CSTNE8M00G55Z000R0, symbol Device:Resonator
- C1: footprint Capacitors_SMD:C_0603 -> Capacitors_SMD:C_0805; #manf UMK107BJ105KA-T -> CL21B105KBFNNNG; order_URL https://www.digikey.jp/product-detail/ja/taiyo-yuden/UMK107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 -> https://www.digikey.jp/product-detail/ja/samsung-electro-me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
- C10: #manf 0603B333K500CT -> 0603YC333KAT2A; order_URL https://www.digikey.jp/product-detail/ja/walsin-technology-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 -> https://www.digikey.jp/product-detail/ja/avx-corporation/06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
- C11: footprint Capacitors_ThroughHole:CP_Radial_D8.0mm_P3.50mm -> 35ZLH220MEFC8X11.5:CP_Radial_D8.0mm_P3.50mm; #manf 35ZLH220MEFCCT8X11.5 -> 35ZLH220MEFC8X11.5; order_URL (none) -> https://akizukidenshi.com/catalog/g/gP-02718/
- C12, C13, C14, C15, C16, C4, C5, C7, C8, C9: #manf C0603C104M4RACTU -> CL10B104KO8NNNC; order_URL https://www.digikey.jp/product-detail/ja/kemet/C0603C104M4R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 -> https://www.digikey.jp/product-detail/ja/samsung-electro-me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
- C17, C18, C19, C20, C21: footprint Capacitors_SMD:C_0603 -> Capacitors_SMD:C_1210; #manf GRM188R6YA106MA73 -> GRM32ER7YA106KA12; order_URL https://akizukidenshi.com/catalog/g/gP-13161/ -> https://akizukidenshi.com/catalog/g/gP-06043/
- C2: #manf CL10A225KQ8NNNC -> CL10B225KP8NFNC; order_URL https://www.digikey.jp/product-detail/ja/samsung-electro-mechanics/CL10A225KQ8NNNC/1276-1183-1-ND/3889269 -> https://www.digikey.jp/product-detail/ja/samsung-electro-mechanics/CL10B225KP8NFNC/1276-2016-1-ND/3890102
- C3: #manf CL10B105MO8NNWC -> CL10B105KP8NNNC; order_URL https://www.digikey.jp/product-detail/ja/samsung-electro-mechanics/CL10B105MO8NNWC/1276-6524-1-ND/5961383 -> https://www.digikey.jp/product-detail/ja/samsung-electro-mechanics/CL10B105KP8NNNC/1276-1946-1-ND/3890032
- C6: #manf 0603B103K500CT -> 0603B103K160CT; order_URL https://www.digikey.jp/product-detail/ja/walsin-technology-corporation/0603B103K500CT/1292-1386-1-ND/9355390 -> https://www.digikey.jp/product-detail/ja/walsin-technology-corporation/0603B103K160CT/1292-1384-1-ND/9355388
- J4: value Conn_01x04 -> 4_SMD_Pad; footprint Pin_Headers:Pin_Header_Straight_1x04_Pitch2.54mm -> SMD_Pad:4_SMD_Pad
- R8: value 1.5k -> 1.5k 1%
Connections:
- net +3V3: now also J10.3 (Pin_3), J11.1 (Pin_1), J12.3 (Pin_3); no longer R1.1, U2.31 (BOOT0)
- net +BATT: now also C22.1, H3.1, J5.4 (Pin_4), J7.4 (Pin_4), J9.2 (Pin_2)
- net CS: now also J6.2 (Pin_2), J8.2 (Pin_2)
- net GND: now also C22.2, H4.1, J10.4 (Pin_4), J11.3 (Pin_3), J12.4 (Pin_4), J5.1 (Pin_1), J6.3 (Pin_3), J7.1 (Pin_1), J8.3 (Pin_3), J9.1 (Pin_1), Y1.2
- net INA: now also J5.3 (Pin_3), J7.3 (Pin_3)
- net INB: now also J5.2 (Pin_2), J7.2 (Pin_2)
- net OUTA: now also H1.1
- net OUTB: now also H2.1
- net PWM: now also J6.1 (Pin_1), J8.1 (Pin_1)
- net Potentiometer: now also J11.2 (Pin_2), J12.5 (Pin_5)
- net RS485_D+: now also J9.3 (Pin_3)
- net RS485_D-: now also J9.4 (Pin_4)
- net SCL: now also J10.1 (Pin_1), J12.1 (Pin_1)
- net SDA: now also J10.2 (Pin_2), J12.2 (Pin_2)
- net SEL0: now also J6.4 (Pin_4), J8.4 (Pin_4)
- net at U2.2 (PF0): now also Y1.1
- net at U2.3 (PF1): now also Y1.3
- new net: R1.1, U2.31 (BOOT0)
- no-connect marks 9 -> 7
Other:
- note added: "35V X7R(-55-125°C ±15%)"
- moved on the sheet: C10, C11, C15, C17, C18, C19, C20, C21, C9, D1, D3, J1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

Commit message: Add files via upload
Parts:
- J10: value Conn_01x04 -> S4B-PH-K; footprint Connect:Grove_1x04 -> Connectors_JST:JST_PH_S4B-PH-K_1x04_P2.00mm_Horizontal
Connections:
- net ENC_A: now also J4.1 (Pin_1), U2.12 (PA6); no longer J4.3 (Pin_3), U2.11 (PA5)
- net ENC_B: now also U2.10 (PA4); no longer U2.26 (PB3)
- net GND: now also J4.3 (Pin_3); no longer J4.1 (Pin_1)
- no-connect marks 7 -> 6
Other:
- note added: "TIM3_CH1"
- note added: "TIM3_CH2"
- note removed: "TIM2_CH1"
- note removed: "TIM2_CH2"
- moved on the sheet: C15, H3, H4, J10, R13, R14, U7

Commit message: fix ver.0.2
Parts:
- C1: #manf CL21B105KBFNNNG -> CL21B105KBFNFNE; order_URL https://www.digikey.jp/product-detail/ja/samsung-electro-mechanics/CL21B105KBFNNNG/1276-6470-1-ND/5958098 -> https://www.digikey.jp/product-detail/ja/samsung-electro-mechanics/CL21B105KBFNFNE/1276-2928-1-ND/3891014
- D2, D3: footprint Diodes_SMD:D_SOD-523 -> Diodes_SMD:D_SOD-323
- J5, J6: #manf (none) -> 2210S-40G; order_URL (none) -> https://akizukidenshi.com/catalog/g/gC-03867/
- R1, R12, R13, R14, R15, R2, R7: #manf ‎RC0603JR-0710KL‎ -> RC0603JR-0710KL
Changed lines of the file:
@@
 F 2 "Resistors_SMD:R_0603" V 10080 2050 50  0001 C CNN
 F 3 "~" H 10150 2050 50  0001 C CNN
-F 4 "‎RC0603JR-0710KL‎" H 10150 2050 50  0001 C CNN "#manf"
+F 4 "RC0603JR-0710KL" H 10150 2050 50  0001 C CNN "#manf"
 F 5 "https://www.digikey.jp/product-detail/ja/yageo/RC0603JR-0710KL/311-10KGRCT-ND/729647" H 10150 2050 50  0001 C CNN "order_URL"
 	1    10150 2050
@@
 F 2 "Resistors_SMD:R_0603" V 3780 3800 50  0001 C CNN
 F 3 "~" H 3850 3800 50  0001 C CNN
-F 4 "‎RC0603JR-0710KL‎" H 3850 3800 50  0001 C CNN "#manf"
+F 4 "RC0603JR-0710KL" H 3850 3800 50  0001 C CNN "#manf"
 F 5 "https://www.digikey.jp/product-detail/ja/yageo/RC0603JR-0710KL/311-10KGRCT-ND/729647" H 3850 3800 50  0001 C CNN "order_URL"
 	1    3850 3800
@@
 F 2 "Resistors_SMD:R_0603" V 7130 3750 50  0001 C CNN
 F 3 "~" H 7200 3750 50  0001 C CNN
-F 4 "‎RC0603JR-0710KL‎" H 7200 3750 50  0001 C CNN "#manf"
+F 4 "RC0603JR-0710KL" H 7200 3750 50  0001 C CNN "#manf"
 F 5 "https://www.digikey.jp/product-detail/ja/yageo/RC0603JR-0710KL/311-10KGRCT-ND/729647" H 7200 3750 50  0001 C CNN "order_URL"
 	1    7200 3750
@@
 F 2 "Capacitors_SMD:C_0805" H 1338 2400 50  0001 C CNN
 F 3 "https://media.digikey.com/pdf/Data%20Sheets/Samsung%20PDFs/CL21B105KBFNNNG_Spec.pdf" H 1300 2550 50  0001 C CNN
-F 4 "CL21B105KBFNNNG" H 1300 2550 50  0001 C CNN "#manf"
-F 5 "https://www.digikey.jp/product-detail/ja/samsung-electro-mechanics/CL21B105KBFNNNG/1276-6470-1-ND/5958098" H 1300 2550 50  0001 C CNN "order_URL"
+F 4 "CL21B105KBFNFNE" H 1300 2550 50  0001 C CNN "#manf"
+F 5 "https://www.digikey.jp/product-detail/ja/samsung-electro-mechanics/CL21B105KBFNFNE/1276-2928-1-ND/3891014" H 1300 2550 50  0001 C CNN "order_URL"
 	1    1300 2550
 	1    0    0    -1
@@
 F 0 "D2" V 3146 7179 50  0000 L CNN
 F 1 "D_TVS" V 3055 7179 50  0000 L CNN
-F 2 "Diodes_SMD:D_SOD-523" H 3100 7100 50  0001 C CNN
+F 2 "Diodes_SMD:D_SOD-323" H 3100 7100 50  0001 C CNN
 F 3 "https://assets.nexperia.com/documents/data-sheet/PESD3V3U1UA_UB_UL.pdf" H 3100 7100 50  0001 C CNN
 F 4 "PESD3V3U1UA,115" V 3100 7100 50  0001 C CNN "#manf"
@@
 F 0 "D3" V 1746 4670 50  0000 R CNN
 F 1 "D_TVS" V 1655 4670 50  0000 R CNN
-F 2 "Diodes_SMD:D_SOD-523" H 1700 4750 50  0001 C CNN
+F 2 "Diodes_SMD:D_SOD-323" H 1700 4750 50  0001 C CNN
 F 3 "https://assets.nexperia.com/documents/data-sheet/PESD3V3U1UA_UB_UL.pdf" H 1700 4750 50  0001 C CNN
 F 4 "PESD3V3U1UA,115" V 1700 4750 50  0001 C CNN "#manf"
@@
 F 2 "Resistors_SMD:R_0603" V 8830 5450 50  0001 C CNN
 F 3 "~" H 8900 5450 50  0001 C CNN
-F 4 "‎RC0603JR-0710KL‎" H 8900 5450 50  0001 C CNN "#manf"
+F 4 "RC0603JR-0710KL" H 8900 5450 50  0001 C CNN "#manf"
 F 5 "https://www.digikey.jp/product-detail/ja/yageo/RC0603JR-0710KL/311-10KGRCT-ND/729647" H 8900 5450 50  0001 C CNN "order_URL"
 	1    8900 5450
@@
 F 2 "Resistors_SMD:R_0603" V 8730 5450 50  0001 C CNN
 F 3 "~" H 8800 5450 50  0001 C CNN
-F 4 "‎RC0603JR-0710KL‎" H 8800 5450 50  0001 C CNN "#manf"
+F 4 "RC0603JR-0710KL" H 8800 5450 50  0001 C CNN "#manf"
 F 5 "https://www.digikey.jp/product-detail/ja/yageo/RC0603JR-0710KL/311-10KGRCT-ND/729647" H 8800 5450 50  0001 C CNN "order_URL"
 	1    8800 5450
@@
 F 2 "Resistors_SMD:R_0603" V 2830 6700 50  0001 C CNN
 F 3 "~" H 2900 6700 50  0001 C CNN
-F 4 "‎RC0603JR-0710KL‎" H 2900 6700 50  0001 C CNN "#manf"
+F 4 "RC0603JR-0710KL" H 2900 6700 50  0001 C CNN "#manf"
 F 5 "https://www.digikey.jp/product-detail/ja/yageo/RC0603JR-0710KL/311-10KGRCT-ND/729647" H 2900 6700 50  0001 C CNN "order_URL"
 	1    2900 6700
@@
 F 2 "Resistors_SMD:R_0603" V 3930 3350 50  0001 C CNN
 F 3 "~" H 4000 3350 50  0001 C CNN
-F 4 "‎RC0603JR-0710KL‎" H 4000 3350 50  0001 C CNN "#manf"
+F 4 "RC0603JR-0710KL" H 4000 3350 50  0001 C CNN "#manf"
 F 5 "https://www.digikey.jp/product-detail/ja/yageo/RC0603JR-0710KL/311-10KGRCT-ND/729647" H 4000 3350 50  0001 C CNN "order_URL"
 	1    4000 3350
@@
 F 2 "Pin_Headers:Pin_Header_Straight_1x04_Pitch2.00mm" H 9600 2900 50  0001 C CNN
 F 3 "" H 9600 2900 50  0001 C CNN
-F 4 "" H 9600 2900 50  0001 C CNN "#manf"
-F 5 "" H 9600 2900 50  0001 C CNN "order_URL"
+F 4 "2210S-40G" H 9600 2900 50  0001 C CNN "#manf"
+F 5 "https://akizukidenshi.com/catalog/g/gC-03867/" H 9600 2900 50  0001 C CNN "order_URL"
 	1    9600 2900
 	1    0    0    1
@@
 F 2 "Pin_Headers:Pin_Header_Straight_1x04_Pitch2.00mm" H 7750 2900 50  0001 C CNN
 F 3 "" H 7750 2900 50  0001 C CNN
-F 4 "" H 7750 2900 50  0001 C CNN "#manf"
-F 5 "" H 7750 2900 50  0001 C CNN "order_URL"
+F 4 "2210S-40G" H 7750 2900 50  0001 C CNN "#manf"
+F 5 "https://akizukidenshi.com/catalog/g/gC-03867/" H 7750 2900 50  0001 C CNN "order_URL"
 	1    7750 2900
 	-1   0    0    1
@@
 Data
 89 50 4E 47 0D 0A 1A 0A 00 00 00 0D 49 48 44 52 00 00 02 C7 00 00 02 5C 08 02 00 00 00 9A 35 9E
-F9 00 00 00 03 73 42 49 54 08 08 08 DB E1 4F E0 00 00 00 09 70 48 59 73 00 00 0E C3 00 00 0E C3
-01 C7 6F A8 64 00 00 20 00 49 44 41 54 78 9C EC 9D 77 B4 64 55 95 FF BF E7 9C 9B 2A BC FC 5E 37
+F9 00 00 00 03 73 42 49 54 08 08 08 DB E1 4F E0 00 00 00 09 70 48 59 73 00 00 0E 74 00 00 0E 74
+01 6B 24 B3 D6 00 00 20 00 49 44 41 54 78 9C EC 9D 77 B4 64 55 95 FF BF E7 9C 9B 2A BC FC 5E 37
 1D E8 6E 82 0D 28 20 02 E3 8C 22 59 5B 30 01 82 8E 08 C2 52 14 66 06 51 74 44 D7 38 8E 4B 58 CA
 A8 88 B8 9C 31 FE 46 1D 03 28 51 40 50 1C 07 14 E6 87 3F 75 48 D2 08 1D E8 1C 5E 8E 15 6F 38 67
